File: docs/kicad/Gap_dipole.kicad_sch (KiCad schematic)
At the start: 30 parts, among them J1 Conn_Coaxial, K1 Nonlatching, K2 Nonlatching, K3 Nonlatching, K4 Nonlatching, K5 Nonlatching, K6 Nonlatching, K7 Nonlatching, U1 REG

Commit message: updates after Bob's review
Parts:
- removed LC_Network: ~, symbol GapDipoleSymbols:Generic_device
- added G1: ~, symbol GapDipoleSymbols:Generic_device
- R1, R2: value R_US -> 100Ω
Connections:
- net GNDREF: now also K1.12, K2.12, K3.12, K4.12, K5.12, K6.1, G1.3 (gnd); no longer K1.4
- net at C1.1, J1.1 (In), K1.9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: now also K1.4
- net at K4.3: now also G1.1 (in)
- net at Balun.2 (AB): now also K4.9; no longer K4.8
- net at K1.10, K3.4: now also K1.3, K3.9
- net at K1.5, K2.4: now also K1.8, K2.9
- net at K3.5, K4.4: now also K3.8; no longer K4.9
- net at K4.10: now also G1.2 (out)
- net at K4.5: now also K4.8
Other:
- note added: ""match" (unenergized)"
- note added: "All "GNDREF" are actually vias to bottom layer of board (ground plane)"
- note added: "RF"
- note added: "Schematic v. board -- notes GNDREF is the groundplane. Will be back copper layer of board. All connections will be using vias to the groundplane layer. Traces here on the schematic are logical. On the pcb the traces will be broad & spaced following RF board design guidelines."
- note removed: ""match""
- note removed: "center"
- note removed: "shield"

Commit message: updated k3 to connect to LC when unenergized
Connections:
- net at R2.1: now also K3.8; no longer K3.10
- net at K3.3: now also K3.10, K4.4; no longer R1.1
- new net: K3.5, R1.1
Other:
- note added: "Relays shown in their unenergized state."
- note removed: "Bias tee"
- moved on the sheet: R1, R2
