File: board/Gap_dipole.kicad_pcb (KiCad board)
At the start: 2 copper layers, 25 parts, among them K1 EE2-3NU, K10 EE2-3SNUH, K11 EE2-3NU, K2 EE2-3NU, K3 EE2-3NU, K4 EE2-3NU, K5 EE2-3NU, K6 EE2-3NU, K8 EE2-3NU, K9 EE2-3SNUH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

Commit message: relay parts are right now
Parts:
- removed K10: EE2-3SNUH, Relay_SMD:Relay_DPDT_Kemet_EE2_NUH
- removed K11: EE2-3NU, Relay_SMD:Relay_DPDT_Kemet_EE2_NU
- added D10: 1N4148WS, Diode_SMD:D_SOD-323, F.Cu at (91.1, 53.0)
- added D11: 1N4148WS, Diode_SMD:D_SOD-323, F.Cu at (91.1, 56.0)
- added D12: 1N4148WS, Diode_SMD:D_SOD-323, F.Cu at (91.1, 58.9)
- added D13: 1N4148WS, Diode_SMD:D_SOD-323, F.Cu at (91.1, 61.9)
- added D7: 1N4148WS, Diode_SMD:D_SOD-323, F.Cu at (91.1, 44.1)
- added D8: 1N4148WS, Diode_SMD:D_SOD-323, F.Cu at (91.1, 47.1)
- added D9: 1N4148WS, Diode_SMD:D_SOD-323, F.Cu at (91.1, 50.0)
- added K7: EE2-3NU, Relay_SMD:Relay_DPDT_Kemet_EE2_NU, F.Cu at (112.0, 34.4)
- added U2: ESP32-S3-DevKitC, Espressif:ESP32-S3-DevKitC, F.Cu at (37.1, 50.2)
- K8: value EE2-3NU -> EE2-3SNUH; footprint Relay_SMD:Relay_DPDT_Kemet_EE2_NU -> Relay_SMD:Relay_DPDT_Kemet_EE2_NUH
- moved L1 84.7 mm to (79.5, 97.4)
- moved R1 80.8 mm to (74.8, 97.5)
- moved R2 80.8 mm to (74.8, 100.4)
- moved C4 74.9 mm to (63.6, 71.7)
- moved C5 74.9 mm to (63.6, 75.8)
- moved C6 74.9 mm to (63.6, 80.0)
- moved C7 74.9 mm to (63.6, 84.2)
- moved D1 74.9 mm to (74.3, 87.2)
- moved L2 74.9 mm to (74.4, 77.9)
- moved L3 74.9 mm to (74.4, 82.7)
- moved C2 74.9 mm to (75.6, 91.0)
- moved C3 74.9 mm to (75.6, 94.3)
- moved U1 74.9 mm to (75.9, 73.5)
- moved K8 70.6 mm to (98.2, 51.0)
- moved K3 63.6 mm to (64.6, 34.4)
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Connections:
- K1 pad 1: unconnected-(K1-Pad1) -> Net-(D7-K)
- K1 pad 10: +3.3V -> Net-(K1-Pad10)
- K1 pad 3: GNDREF -> Net-(K1-Pad10)
- K1 pad 4: Net-(K1-Pad4) -> Net-(C1-Pad1)
- K1 pad 5: +3.3V -> Net-(K1-Pad5)
- K1 pad 8: GNDREF -> Net-(K1-Pad5)
- K1 pad 9: Net-(K1-Pad9) -> Net-(C1-Pad1)
- K2 pad 1: unconnected-(K2-Pad1) -> Net-(D8-K)
- K2 pad 4: Net-(K2-Pad4) -> Net-(K1-Pad10)
- K2 pad 9: Net-(K2-Pad4) -> Net-(K1-Pad10)
- K3 pad 1: unconnected-(K3-Pad1) -> Net-(D10-K)
- K3 pad 10: Net-(K2-Pad4) -> Net-(K3-Pad10)
- K3 pad 3: Net-(K2-Pad4) -> Net-(K3-Pad3)
- K3 pad 4: Net-(C1-Pad1) -> Net-(K1-Pad5)
- K3 pad 9: Net-(C1-Pad1) -> Net-(K1-Pad5)
- K4 pad 1: unconnected-(K4-Pad1) -> Net-(D9-K)
- K4 pad 3: Net-(K4-Pad3) -> Net-(K4-Pad10)
- K4 pad 4: Net-(K3-Pad5) -> Net-(Balun1-AB)
- K4 pad 8: Net-(K4-Pad5) -> Net-(K4-Pad8)
- K5 pad 1: unconnected-(K5-Pad1) -> Net-(D11-K)
- K5 pad 5: Net-(K1-Pad4) -> Net-(K5-Pad5)
- K5 pad 8: Net-(K1-Pad9) -> Net-(K5-Pad8)
- K6 pad 1: unconnected-(K6-Pad1) -> GNDREF
- K6 pad 10: unconnected-(K6-Pad10) -> Net-(Balun1-SA)
- K6 pad 12: unconnected-(K6-Pad12) -> Net-(D13-K)
- K6 pad 3: unconnected-(K6-Pad3) -> Net-(Balun1-SA)
- K6 pad 4: unconnected-(K6-Pad4) -> Net-(K6-Pad4)
- K6 pad 5: unconnected-(K6-Pad5) -> Net-(K5-Pad5)
- K6 pad 8: unconnected-(K6-Pad8) -> Net-(K5-Pad8)
- K6 pad 9: unconnected-(K6-Pad9) -> Net-(K6-Pad9)
- K8 pad 1: unconnected-(K8-Pad1) -> Net-(C5-Pad1)
- K8 pad 10: Net-(K8-Pad10) -> unconnected-(K8-Pad10)
- K8 pad 12: GNDREF -> Net-(C5-Pad2)
- K8 pad 3: Net-(K8-Pad10) -> unconnected-(K8-Pad3)
- K8 pad 4: Net-(Balun1-AB) -> Net-(C5-Pad2)
- K8 pad 5: Net-(K8-Pad5) -> Net-(C4-Pad2)
- K8 pad 8: Net-(K8-Pad8) -> Net-(C4-Pad1)
- K8 pad 9: Net-(K4-Pad5) -> Net-(C5-Pad1)
- K9 pad 1: Net-(C5-Pad1) -> Net-(C7-Pad1)
- K9 pad 12: Net-(C5-Pad2) -> Net-(C7-Pad2)
- K9 pad 4: Net-(C5-Pad2) -> Net-(C7-Pad2)
- K9 pad 5: Net-(C4-Pad2) -> Net-(C6-Pad2)
- K9 pad 8: Net-(C4-Pad1) -> Net-(C6-Pad1)
- K9 pad 9: Net-(C5-Pad1) -> Net-(C7-Pad1)
- R1 pad 1: Net-(K4-Pad10) -> Net-(K3-Pad10)
- R2 pad 1: Net-(K4-Pad3) -> Net-(K3-Pad3)
