File: board/Gap_dipole.kicad_sch (KiCad schematic)
At the start: 79 parts, among them K1 Nonlatching, K2 Nonlatching, K3 Nonlatching, K4 Nonlatching, sweep (energized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, K5 Nonlatching, K6 Nonlatching, K7 Nonlatching, K8 Relay_DPDT_Latching_1coil (bi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, U1 REG

Commit message: replaced generic relays with specific parts with footprints, added diodes for relays, cleanup
Parts:
- removed C10, C11, C12, C13, C14, C15, C8, C9: C, Capacitor_THT:C_Disc_D7.0mm_W2.5mm_P5.00mm, symbol Device:C
- removed D10, D11, D12, D13, D14, D15, D16, D17, D2, D3, D4, D5, D6, D7, D8, D9: D, Diode_SMD:D_0805_2012Metric_Pad1.15x1.40mm_HandSolder, symbol Device:D
- removed K1, K2, K3, K5, K6, K7: Nonlatching, Relay_THT:Relay_DPDT_Kemet_EC2_NU, symbol Relay:EC2-3NU
- removed K4: Nonlatching, sweep (energized) or match (unenergi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, Relay_THT:Relay_DPDT_Kemet_EC2_NU, symbol Relay:EC2-3NU
- removed K8: Relay_DPDT_Latching_1coil (bipolar) sets shunt si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, Relay_THT:Relay_DPDT_Kemet_EC2_NJ, symbol Relay:Relay_DPDT_Latching_1coil
- removed KC1, KC2, KC3, KC4, KC5, KC6, KC7, KC8, KL1, KL2, KL3, KL4, KL5, KL6, KL7, KL8, KLB1, KLB2: Relay_DPDT_Latching_1coil (bipolar), Relay_THT:Relay_DPDT_Kemet_EC2_NJ, symbol Relay:Relay_DPDT_Latching_1coil
- removed L10, L4, L5, L6, L7, L8, L9: L, Inductor_THT:L_Toroid_Vertical_L10.0mm_W5.0mm_P5.08mm, symbol Device:L
- removed L11: L, Inductor_THT:L_Toroid_Horizontal_D12.7mm_P20.00mm_Diameter14-5mm_Amidon-T50, symbol Device:L
- added D10, D11, D12, D13, D2, D3, D4, D5, D6, D7, D8, D9: 1N4148WS, Diode_SMD:D_SOD-323, symbol Diode:1N4148WS
- added K1, K2, K3, K4, K5 (x2), K7: EE2-3NU, Relay_SMD:Relay_DPDT_Kemet_EE2_NU, symbol Relay:EE2-3NU
- added K8, K9: EE2-3SNUH, Relay_SMD:Relay_DPDT_Kemet_EE2_NUH, symbol Relay:EE2-3SNUH
Connections:
- net +3.3V: now also K7.10, K7.5
- net GNDREF: now also D10.2 (A), D11.2 (A), D12.2 (A), D13.2 (A), D2.2 (A), D3.2 (A), D4.2 (A), D5.2 (A), D6.2 (A), D7.2 (A), D8.2 (A), D9.2 (A), K1.12, K2.10, K2.12, K2.3, K3.12, K4.12, K5.1, K5.12, K7.12, K7.3, K7.8
- net at R2.1: now also K3.3
- net at C1.1, JC1.1 (In), L1.1: now also K1.4, K1.9
- net at C4.1: now also K8.8
- net at C4.2: now also K8.5
- net at G1.1 (in): now also K4.8
- net at G1.2 (out): now also K4.5
- net at Banana4.1, C7.2, L3.2: now also K9.12, K9.4
- net at Banana4.2: now also K5.4
- net at Banana1.1, C5.1, L2.1: now also K8.1, K8.9
- net at Banana2.1, C5.2, L2.2: now also K8.12, K8.4
- net at Banana3.1, C7.1, L3.1: now also K9.1, K9.9
- net at R1.1: now also K3.10
- net at Banana1.2: now also K5.9
- net at Balun1.3 (SA): now also K5.10, K5.3
- net at Banana3.2: now also K5.9
- net at Balun1.2 (AB): now also K4.4
- net at Balun1.4 (SB): now also K5.10, K5.3
- net at C6.2: now also K9.5
- net at C6.1: now also K9.8
- net at Banana2.2: now also K5.4
- new net: D10.1 (K), K3.1
- new net: D8.1 (K), K2.1
- new net: K1.10, K1.3, K2.4, K2.9
- new net: D7.1 (K), K1.1
- new net: K1.5, K1.8, K3.4, K3.9
- new net: D9.1 (K), K4.1
- new net: K4.10, K4.3
- new net: K3.5, K3.8, K4.9
- new net: D13.1 (K), K5.12
- new net: K5.5, K5.5, K7.4
- new net: K5.8, K5.8, K7.9
- new net: D12.1 (K), K7.1
- new net: D11.1 (K), K5.1

Commit message: relay parts are right now
Parts:
- removed D2, D3, D4, D5, D6: 1N4148WS, Diode_SMD:D_SOD-323, symbol Diode:1N4148WS
- added U2: ESP32-S3-DevKitC, Espressif:ESP32-S3-DevKitC, symbol Espressif:ESP32-S3-DevKitC
- renumbered K5 to K6
Connections:
- new net: U2.1 (3V3), U2.2 (3V3)
- new net: U2.22 (GND), U2.23 (GND), U2.24 (GND), U2.44 (GND)
Other:
- note added: "Esprsssif ESP32-S3-DevkitC"
